File: TH-XWhatsIt/model f plugboard.sch (KiCad schematic (older format))
At the start: 3 parts, among them J3 MODEL F PLUGBOARD COLUMNS, J4 MODEL F PLUGBOARD CONNECTOR, J5 MODEL F PLUGBOARD ROWS

Commit message: version bump to 2.0 due to header position changes finished wiring up most of the plugboards, but displaywriter as per usual is the most annoying.....see changes file for more details (jan 3rd, 2020)
Connections:
- net MFSENSE1: now also J5.10 (Pin_10); no longer J5.3 (Pin_3)
- net MFSENSE2: now also J5.9 (Pin_9); no longer J5.4 (Pin_4)
- net MFSENSE3: now also J5.8 (Pin_8); no longer J5.5 (Pin_5)
- net MFSENSE4: now also J5.7 (Pin_7); no longer J5.6 (Pin_6)
- net MFSENSE5: now also J5.6 (Pin_6); no longer J5.7 (Pin_7)
- net MFSENSE6: now also J5.5 (Pin_5); no longer J5.8 (Pin_8)
- net MFSENSE7: now also J5.4 (Pin_4); no longer J5.9 (Pin_9)
- net MFSENSE8: now also J5.3 (Pin_3); no longer J5.10 (Pin_10)
Changed lines of the file:
@@
 EESchema Schematic File Version 4
+LIBS:TH-XWhatsIt-cache
 EELAYER 30 0
 EELAYER END
@@
 Text HLabel 5200 3050 0    50   Input ~ 0
 MFCOL16
+Text HLabel 2850 5200 0    50   BiDi ~ 0
+MFSENSE1
+Text HLabel 2850 5100 0    50   BiDi ~ 0
+MFSENSE2
+Text HLabel 2850 5000 0    50   BiDi ~ 0
+MFSENSE3
+Text HLabel 2850 4900 0    50   BiDi ~ 0
+MFSENSE4
+Text HLabel 2850 4800 0    50   BiDi ~ 0
+MFSENSE5
+Text HLabel 2850 4700 0    50   BiDi ~ 0
+MFSENSE6
+Text HLabel 2850 4600 0    50   BiDi ~ 0
+MFSENSE7
 Text HLabel 2850 4500 0    50   BiDi ~ 0
-MFSENSE1
-Text HLabel 2850 4600 0    50   BiDi ~ 0
-MFSENSE2
-Text HLabel 2850 4700 0    50   BiDi ~ 0
-MFSENSE3
-Text HLabel 2850 4800 0    50   BiDi ~ 0
-MFSENSE4
-Text HLabel 2850 4900 0    50   BiDi ~ 0
-MFSENSE5
-Text HLabel 2850 5000 0    50   BiDi ~ 0
-MFSENSE6
-Text HLabel 2850 5100 0    50   BiDi ~ 0
-MFSENSE7
-Text HLabel 2850 5200 0    50   BiDi ~ 0
 MFSENSE8
 Text HLabel 5200 3350 0    50   BiDi ~ 0

Commit message: finished wiring the dispalywriter plugboard, and added grounding straps to plugboards
Parts:
- added H2: GROUND STRAP, MountingHole:MountingHole_2.2mm_M2_Pad_Via, symbol Mechanical:MountingHole_Pad
Connections:
- net MFGROUND: now also H2.1
Changed lines of the file:
@@
 Text Notes 3950 7750 0    50   ~ 0
 Copyright Rainy Day Plans.\nThis documentation describes Open Hardware and is licensed under the\nCERN OHL v. 1.2.\nYou may redistribute and modify this documentation under the terms of the\nCERN OHL v.1.2. (http://ohwr.org/cernohl). This documentation is distributed\nWITHOUT ANY EXPRESS OR IMPLIED WARRANTY, INCLUDING OF\nMERCHANTABILITY, SATISFACTORY QUALITY AND FITNESS FOR A\nPARTICULAR PURPOSE. Please see the CERN OHL v.1.2 for applicable\nconditions
+$Comp
+L Mechanical:MountingHole_Pad H2
+U 1 1 5E39F8A0
+P 5200 4950
+F 0 "H2" H 5300 4999 50  0000 L CNN
+F 1 "GROUND STRAP" H 5300 4908 50  0000 L CNN
+F 2 "MountingHole:MountingHole_2.2mm_M2_Pad_Via" H 5200 4950 50  0001 C CNN
+F 3 "~" H 5200 4950 50  0001 C CNN
+	1    5200 4950
+	1    0    0    -1
+$EndComp
+Text HLabel 5200 5050 3    50   UnSpc ~ 0
+MFGROUND
 $EndSCHEMATC

Commit message: initial update to switch to smd, so now th prefix is a misnomer
Parts:
- H2: footprint MountingHole:MountingHole_2.2mm_M2_Pad_Via -> MountingHole:MountingHole_3mm_Pad_Via
Changed lines of the file:
@@
 F 0 "H2" H 5300 4999 50  0000 L CNN
 F 1 "GROUND STRAP" H 5300 4908 50  0000 L CNN
-F 2 "MountingHole:MountingHole_2.2mm_M2_Pad_Via" H 5200 4950 50  0001 C CNN
+F 2 "MountingHole:MountingHole_3mm_Pad_Via" H 5200 4950 50  0001 C CNN
 F 3 "~" H 5200 4950 50  0001 C CNN
 	1    5200 4950
