File: TH-XWhatsIt/beamspring plugboard.sch (KiCad schematic (older format))
At the start: 5 parts, among them J6 BEAMSPRING PLUGBOARD COLUMNS, J7 BEAMSPRING PLUGBOARD CONNECTOR, J8 BEAMSPRING PLUGBOARD ROWS

Commit message: Added beamspring mounting hole
Parts:
- H5: footprint TH-XWhatsIt:BeamSpringGroundingMountingHole -> TH-XWhatsIt:BeamSpringGroundingMountingHoleForTHOnly
Changed lines of the file:
@@
 F 0 "H5" H 6350 4724 50  0000 L CNN
 F 1 "GROUND STRAP" H 6350 4633 50  0000 L CNN
-F 2 "TH-XWhatsIt:BeamSpringGroundingMountingHole" H 6250 4675 50  0001 C CNN
+F 2 "TH-XWhatsIt:BeamSpringGroundingMountingHoleForTHOnly" H 6250 4675 50  0001 C CNN
 F 3 "~" H 6250 4675 50  0001 C CNN
 	1    6250 4675

Commit message: Various changes to revision 0.1.1
General:
    Made mounting hole bigger (M3). And moved it a little bit so it doesn't interfere with some components.
    Star ground turned into single ground.
    Ground fills added everywhere.
    Many stitching vias added everywhere.
    Added JLCJLCJLCJLC magic string under pro micro. When ordering from JLCPCB, you can select for Order Number: "Specify Location"
    Bumped version number to 0.1.1
    Added silkscreen to mark rows/columns everywhere.
    Added optional holes for soldering grounding wires everywhere.
Controller:
    Added silkscreen to ease debugging, by marking various important nets.
    Rearranged some traces to maintain better separation between traces, and better ground reference.
Model F plugboard:
    Modified 3.96mm pitch holes, to hole sizes and pad sizes that match original xwhatsit model F controller
    Moved 3.96mm pitch holes closer to the edge, so it doesn't interfere with case in F AT cases.
    Added mounting holes
    Added holes to support 3178 keyboards.
Displaywriter:
    Addes support for more connector types. (The displaywriter daughterboard is now taller)
Beamspring:
    Bugfix to a mistake that only affected people that ran update footprints from library.
Beamship daughterboard:
    Added support for more connectors. Added breakoff-able mounting hole.
Parts:
- added H8: Solderable ground strap, TH-XWhatsIt:ChassisGnd, symbol Mechanical:MountingHole_Pad
- H3: value GROUND STRAP -> Grounded hole for M3 standoff; footprint MountingHole:MountingHole_2.2mm_M2_Pad_Via -> MountingHole:MountingHole_3.2mm_M3_Pad_Via
- H5: value GROUND STRAP -> Beamspring Mounting Hole
Connections:
- net BSGROUND: now also H8.1
Other:
- moved on the sheet: H5
Changed lines of the file:
@@
 P 5150 4675
 F 0 "H3" H 5250 4724 50  0000 L CNN
-F 1 "GROUND STRAP" H 5250 4633 50  0000 L CNN
-F 2 "MountingHole:MountingHole_2.2mm_M2_Pad_Via" H 5150 4675 50  0001 C CNN
+F 1 "Grounded hole for M3 standoff" H 5250 4633 50  0000 L CNN
+F 2 "MountingHole:MountingHole_3.2mm_M3_Pad_Via" H 5150 4675 50  0001 C CNN
 F 3 "~" H 5150 4675 50  0001 C CNN
 	1    5150 4675
@@
 L Mechanical:MountingHole_Pad H5
 U 1 1 5F892130
-P 6250 4675
-F 0 "H5" H 6350 4724 50  0000 L CNN
-F 1 "GROUND STRAP" H 6350 4633 50  0000 L CNN
-F 2 "TH-XWhatsIt:BeamSpringGroundingMountingHoleForTHOnly" H 6250 4675 50  0001 C CNN
-F 3 "~" H 6250 4675 50  0001 C CNN
-	1    6250 4675
+P 6000 5025
+F 0 "H5" H 6100 5074 50  0000 L CNN
+F 1 "Beamspring Mounting Hole" H 6100 4983 50  0000 L CNN
+F 2 "TH-XWhatsIt:BeamSpringGroundingMountingHoleForTHOnly" H 6000 5025 50  0001 C CNN
+F 3 "~" H 6000 5025 50  0001 C CNN
+	1    6000 5025
 	1    0    0    -1
 $EndComp
-Text HLabel 6250 4775 3    50   UnSpc ~ 0
+Text HLabel 6000 5125 3    50   UnSpc ~ 0
+BSGROUND
+$Comp
+L Mechanical:MountingHole_Pad H8
+U 1 1 5FBD52CB
+P 6925 5475
+F 0 "H8" H 7025 5524 50  0000 L CNN
+F 1 "Solderable ground strap" H 7025 5433 50  0000 L CNN
+F 2 "TH-XWhatsIt:ChassisGnd" H 6925 5475 50  0001 C CNN
+F 3 "~" H 6925 5475 50  0001 C CNN
+	1    6925 5475
+	1    0    0    -1
+$EndComp
+Text HLabel 6925 5575 3    50   UnSpc ~ 0
 BSGROUND
 $EndSCHEMATC
